File: shields/387SX_V2/kicad/arduino_387SX_V2.kicad_pcb (KiCad board)
At the start: 4 copper layers, 71.8 x 56.5 mm, 20 parts, among them J2 JTAG, J3 Conn_01x04_Pin

Commit message: Fixed oversight of I2C SDA and SCK pull-up resistors; rearranged EEPROM IC to accommodate.
Parts:
- moved C16 0.33 mm to (180.2, 83.8)
Routing:
- net GND: track 40.6 -> 30.8 mm
- net +3.3VP: track 79.2 -> 76.7 mm
Other:
- board text added: "Revision 4.0 ©2025"
- board text removed: "Revision 3.0 ©2025"
Changed lines of the file:
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@@
 	(footprint "Capacitor_SMD:C_0603_1608Metric_Pad1.08x0.95mm_HandSolder"
 		(layer "F.Cu")
-		(at 180.519622 83.628403 -135)
+		(at 180.23012 83.77988 -135)
 		(descr "Capacitor SMD 0603 (1608 Metric), square (rectangular) end terminal, IPC_7351 nominal with elongated pad for handsoldering. (Body size source: IPC-SM-782 page 76, https://www.pcb-3d.com/wordpress/wp-content/uploads/ipc-sm-782a_amendment_1_and_2.pdf), generated with kicad-footprint-generator")
 		(tags "capacitor handsolder")
 		(property "Reference" "C16"
-			(at -0.000474 -1.483229 225)
+			(at 0 0.73 45)
+			(unlocked yes)
 			(layer "F.SilkS")
 			(effects
 				(font
-					(size 1 1)
+					(size 0.8 0.8)
 					(thickness 0.15)
 				)
+				(justify bottom)
 			)
 		)
@@
 		(tags "capacitor handsolder")
 		(property "Reference" "C28"
-			(at 0.100894 -1.484902 225)
+			(at 0 0.73 45)
+			(unlocked yes)
 			(layer "F.SilkS")
 			(effects
 				(font
-					(size 1 1)
+					(size 0.8 0.8)
 					(thickness 0.15)
 				)
+				(justify bottom)
 			)
 		)
@@
 		(end 204.075741 124.46)
 		(stroke
+			(width 0.15)
+			(type default)
+		)
+		(fill no)
+		(layer "Cmts.User")
+	)
+	(gr_rect
+		(start 132.267534 67.934788)
+		(end 204.075741 124.46)
+		(stroke
 			(width 0.1)
 			(type solid)
@@
 		)
 	)
-	(gr_text "Revision 3.0 ©2025"
+	(gr_text "Revision 4.0 ©2025"
 		(at 137.866524 110.926126 90)
 		(layer "F.SilkS")
@@
 	)
 	(segment
-		(start 181.129502 83.018523)
-		(end 181.598025 82.55)
-		(width 0.25)
-		(layer "F.Cu")
-		(net 6)
-	)
-	(segment
 		(start 149.239485 87.972117)
 		(end 148.915329 87.647961)
@@
 	)
 	(segment
-		(start 174.814922 74.631969)
-		(end 173.720387 75.726504)
-		(width 0.25)
-		(layer "F.Cu")
-		(net 6)
-	)
-	(segment
 		(start 151.4668 107.067717)
 		(end 151.4668 107.014459)
@@
 	)
 	(segment
-		(start 175.028501 74.631969)
-		(end 174.814922 74.631969)
-		(width 0.25)
-		(layer "F.Cu")
-		(net 6)
-	)
-	(segment
 		(start 150.348999 108.185518)
 		(end 151.4668 107.067717)
@@
 	)
 	(segment
-		(start 181.598025 82.55)
-		(end 182.88 82.55)
-		(width 0.25)
-		(layer "F.Cu")
-		(net 6)
-	)
-	(segment
 		(start 188.784252 105.325506)
 		(end 189.047697 105.325506)
@@
 	)
 	(via
-		(at 175.028501 74.631969)
+		(at 173.720387 75.726504)
 		(size 0.8)
 		(drill 0.4)
@@
 	)
 	(via
-		(at 182.88 82.55)
-		(size 0.8)
-		(drill 0.4)
+		(at 180.84 83.17)
+		(size 0.6)
+		(drill 0.3)
 		(layers "F.Cu" "B.Cu")
 		(free yes)
@@
 	)
 	(segment
-		(start 165.915124 81.846782)
-		(end 167.621483 80.140423)
-		(width 0.25)
-		(layer "In2.Cu")
-		(net 6)
-	)
-	(segment
-		(start 165.915124 83.732525)
-		(end 165.915124 81.846782)
-		(width 0.25)
-		(layer "In2.Cu")
-		(net 6)
-	)
-	(segment
-		(start 167.621483 80.140423)
-		(end 169.507226 80.140423)
-		(width 0.25)
-		(layer "In2.Cu")
-		(net 6)
-	)
-	(segment
 		(start 184.084238 96.52)
 		(end 185.42 96.52)
@@
 	)
 	(segment
-		(start 179.909742 84.238283)
-		(end 176.823397 87.324628)
-		(width 0.25)
+		(start 179.62024 84.395819)
+		(end 176.691431 87.324628)
+		(width 1)
 		(layer "F.Cu")
 		(net 60)
@@
 	)
 	(segment
-		(start 157.488832 85.819628)
-		(end 158.372793 84.935667)
-		(width 0.25)
+		(start 177.193806 81.969385)
+		(end 179.62024 84.395819)
+		(width 1)
 		(layer "F.Cu")
 		(net 60)
 	)
 	(segment
-		(start 176.823397 87.324628)
-		(end 176.691431 87.324628)
+		(start 157.488832 85.819628)
+		(end 158.372793 84.935667)
 		(width 0.25)
 		(layer "F.Cu")
@@
 	)
 	(segment
+		(start 177.193806 77.459017)
+		(end 177.193806 81.969385)
+		(width 1)
+		(layer "F.Cu")
+		(net 60)
+	)
+	(segment
 		(start 171.130699 79.194372)
 		(end 171.130699 78.316192)
@@
 	)
 	(segment
+		(start 179.62024 84.38976)
+		(end 179.62024 84.395819)
+		(width 0.25)
+		(layer "F.Cu")
+		(net 60)
+	)
+	(segment
 		(start 153.198334 90.881161)
 		(end 153.262856 90.816639)
@@
 	)
 	(segment
-		(start 176.691431 87.324628)
-		(end 176.691431 85.420291)
-		(width 0.4)
-		(layer "In1.Cu")
-		(net 60)
-	)
-	(segment
-		(start 176.691431 85.420291)
-		(end 177.178956 84.932766)
-		(width 0.4)
-		(layer "In1.Cu")
-		(net 60)
-	)
-	(segment
 		(start 162.323021 108.877242)
 		(end 164.153408 108.877242)
@@
 	)
 	(segment
-		(start 177.178956 84.932766)
-		(end 177.178956 77.473867)
-		(width 0.4)
-		(layer "In1.Cu")
-		(net 60)
-	)
-	(segment
 		(start 164.119073 85.528577)
 		(end 167.711174 85.528577)
@@
 		(hatch edge 0.5)
 		(priority 1)
-		(connect_pads
+		(connect_pads yes
 			(clearance 0.508)
 		)
@@
 				(xy 167.18393 117.880323) (xy 145.715506 96.195712) (xy 167.680095 74.211732) (xy 189.784454 96.223409)
 				(xy 176.882189 109.02261) (xy 174.839555 107.127796) (xy 185.598138 96.304731) (xy 167.844192 78.441237)
-				(xy 149.710553 96.266654) (xy 166.876361 113.335206) (xy 171.230045 108.879196) (xy 172.691521 110.151667)
+				(xy 149.710553 96.266654) (xy 167.744294 114.203139) (xy 174.84 107.12) (xy 176.88 109.02) (xy 176.88 110.22)
 				(xy 181.701404 110.216799)
 			)
@@
 		(layer "In2.Cu")
 		(hatch edge 0.5)
-		(connect_pads
+		(connect_pads yes
 			(clearance 0.508)
 		)
